Commit message: made huge changes, using mtc moveit, updated massively the dashboard for batch weighing, condor integration working, its completely different than the main branch

File: src/niryo_robot_description/urdf/ned3pro/niryo_ned3pro.urdf.xacro (robot description, xacro)
@@ -187,7 +187,7 @@
         </inertial>
         <visual>
-            <origin xyz="0 -0.038 -0.03" rpy="0 0 0" />
-            <geometry>
-                <mesh filename="file://$(find niryo_robot_description)/meshes/ned3pro/stl/scoop_link.STL" scale="0.001 0.001 0.001" />
+            <origin xyz="0 -0.0 -0.0" rpy="0 0 0" />
+            <geometry>
+                <mesh filename="file://$(find niryo_robot_description)/meshes/ned3pro/stl/niryo_scoop-ros.STL" scale="0.001 0.001 0.001" />
             </geometry>
             <material name="tool_color" />
@@ -196,5 +196,5 @@
             <origin xyz="0 0 0" rpy="0 0 0" />
             <geometry>
-                <mesh filename="file://$(find niryo_robot_description)/meshes/ned3pro/stl/scoop_link.STL" scale="0.001 0.001 0.001" />
+                <mesh filename="file://$(find niryo_robot_description)/meshes/ned3pro/stl/niryo_scoop-ros.STL" scale="0.001 0.001 0.001" />
             </geometry>
         </collision>
@@ -266,5 +266,5 @@
         <parent link="hand_link" />
         <child link="tool_link" />
-        <origin xyz="0 0 0" rpy="${PI} -${PI/2} 0" />
+        <origin xyz="0 0 0" rpy="${PI} 0 0" />
     </joint>
     <joint name="joint_led_ring" type="fixed">

Commit message: changes before a new feature of parameterized template scooping

File: src/niryo_robot_description/urdf/ned3pro/niryo_ned3pro.urdf.xacro (robot description, xacro)
@@ -187,5 +187,5 @@
         </inertial>
         <visual>
-            <origin xyz="0 -0.0 -0.0" rpy="0 0 0" />
+            <origin xyz="0.00 -0.0 -0.0" rpy="0 0 0" />
             <geometry>
                 <mesh filename="file://$(find niryo_robot_description)/meshes/ned3pro/stl/niryo_scoop-ros.STL" scale="0.001 0.001 0.001" />
@@ -200,4 +200,5 @@
         </collision>
     </link>
+    <link name="tcp_link" />
     <!-- Joints -->
     <joint name="joint_world" type="fixed">
@@ -266,5 +267,10 @@
         <parent link="hand_link" />
         <child link="tool_link" />
-        <origin xyz="0 0 0" rpy="${PI} 0 0" />
+        <origin xyz="0.00 0 0.043" rpy="${PI} 0 0" />
+    </joint>
+    <joint name="tool_tcp_joint" type="fixed">
+        <parent link="tool_link" />
+        <child link="tcp_link" />
+        <origin xyz="0.183 0 -0.072" rpy="0 0 0" />
     </joint>
     <joint name="joint_led_ring" type="fixed">

Commit message: sim docker created

File: src/niryo_robot_description/urdf/ned3pro/niryo_ned3pro.urdf.xacro (robot description, xacro)
@@ -189,5 +189,5 @@
             <origin xyz="0.00 -0.0 -0.0" rpy="0 0 0" />
             <geometry>
-                <mesh filename="file://$(find niryo_robot_description)/meshes/ned3pro/stl/niryo_scoop-ros.STL" scale="0.001 0.001 0.001" />
+                <mesh filename="file://$(find niryo_robot_description)/meshes/ned3pro/stl/niryo_scoop_v4-ros.STL" scale="0.001 0.001 0.001" />
             </geometry>
             <material name="tool_color" />
@@ -196,5 +196,5 @@
             <origin xyz="0 0 0" rpy="0 0 0" />
             <geometry>
-                <mesh filename="file://$(find niryo_robot_description)/meshes/ned3pro/stl/niryo_scoop-ros.STL" scale="0.001 0.001 0.001" />
+                <mesh filename="file://$(find niryo_robot_description)/meshes/ned3pro/stl/niryo_scoop_v4-ros.STL" scale="0.001 0.001 0.001" />
             </geometry>
         </collision>
@@ -272,5 +272,5 @@
         <parent link="tool_link" />
         <child link="tcp_link" />
-        <origin xyz="0.183 0 -0.072" rpy="0 0 0" />
+        <origin xyz="0.15825 0 -0.09356" rpy="0 0 0" />
     </joint>
     <joint name="joint_led_ring" type="fixed">

File: src/niryo_robot_moveit_interface/config/niryo_ned3pro.urdf (robot description, URDF)
Before this commit: robot niryo_ned3pro, 11 links, 10 joints
Joints:
- joint tool_tcp_joint: origin xyz=0.183 0 -0.072 rpy=0 0 0 -> xyz=0.15825 0 -0.09356 rpy=0 0 0
