Commit message: Add cell-layout module, bench authoring loop, and lighter Ned3pro meshes.
Introduce versioned config/layouts with hot-reload via cell_layout_manager,
mode→layout apply on runtime switch, provenance-gated scoop poses, BT
VerifyCellLayout, and rebuild-free push_layout. Laptop bench uses mock
hardware on ROS_DOMAIN_ID=42; arm authoring uses exclusive scooping_stack
handoff. Decimate Ned3pro visual STLs and switch collisions to AABB boxes
to cut RViz/MoveIt cost; Fleet Console surfaces active layout id/hash.

Co-authored-by: Cursor <cursoragent@cursor.com>

File: src/niryo_ned_moveit_configs/niryo_ned3pro_moveit_config/config/niryo_ned3pro.urdf.xacro (robot description, xacro)
@@ -3,5 +3,5 @@
     <xacro:arg name="initial_positions_file" default="initial_positions.yaml" />
     <!-- Import niryo_ned3pro urdf file -->
-    <xacro:include filename="$(find niryo_ned_description)/urdf/ned3pro/niryo_ned3pro.urdf.xacro" />
+    <xacro:include filename="$(find niryo_robot_description)/urdf/ned3pro/niryo_ned3pro.urdf.xacro" />
     <!-- Import control_xacro -->
     <xacro:include filename="niryo_ned3pro.ros2_control.xacro" />

File: src/niryo_robot_description/urdf/ned3pro/niryo_ned3pro.urdf.xacro (robot description, xacro)
@@ -45,7 +45,7 @@
         </visual>
         <collision>
-            <origin xyz="0 0 0" rpy="0 0 0" />
-            <geometry>
-                <mesh filename="file://$(find niryo_robot_description)/meshes/ned3pro/stl/base_link.STL" />
+            <origin xyz="-0.00220529 -3.22461e-05 0.0504" rpy="0 0 0" />
+            <geometry>
+                <box size="0.189611 0.1816 0.1008" />
             </geometry>
         </collision>
@@ -68,7 +68,7 @@
         </visual>
         <collision>
-            <origin xyz="0 0 0" rpy="0 0 0" />
-            <geometry>
-                <mesh filename="file://$(find niryo_robot_description)/meshes/ned3pro/stl/shoulder_link.STL" />
+            <origin xyz="-0.0217268 0.0065 0.0697806" rpy="0 0 0" />
+            <geometry>
+                <box size="0.175346 0.145 0.141161" />
             </geometry>
         </collision>
@@ -89,7 +89,7 @@
         </visual>
         <collision>
-            <origin xyz="0 0 0" rpy="0 0 ${PI}" />
-            <geometry>
-                <mesh filename="file://$(find niryo_robot_description)/meshes/ned3pro/stl/arm_link.STL" />
+            <origin xyz="-0.00402863 -0.113297 -0.0135" rpy="0 0 ${PI}" />
+            <geometry>
+                <box size="0.103593 0.321803 0.128" />
             </geometry>
         </collision>
@@ -110,7 +110,7 @@
         </visual>
         <collision>
-            <origin xyz="0 0 0" rpy="${PI} 0 ${-PI/2}" />
-            <geometry>
-                <mesh filename="file://$(find niryo_robot_description)/meshes/ned3pro/stl/elbow_link.STL" />
+            <origin xyz="0.008625 -0.0137681 -0.00355" rpy="${PI} 0 ${-PI/2}" />
+            <geometry>
+                <box size="0.09775 0.107964 0.0691" />
             </geometry>
         </collision>
@@ -131,7 +131,7 @@
         </visual>
         <collision>
-            <origin xyz="0 0 0" rpy="${PI} 0 0" />
-            <geometry>
-                <mesh filename="file://$(find niryo_robot_description)/meshes/ned3pro/stl/forearm_link.STL" />
+            <origin xyz="9.31323e-10 -0.0149 -0.1563" rpy="${PI} 0 0" />
+            <geometry>
+                <box size="0.054 0.0942 0.217815" />
             </geometry>
         </collision>
@@ -152,7 +152,7 @@
         </visual>
         <collision>
-            <origin xyz="0 0 0" rpy="0 0 ${PI/2}" />
-            <geometry>
-                <mesh filename="file://$(find niryo_robot_description)/meshes/ned3pro/stl/wrist_link.STL" />
+            <origin xyz="0.0205 0.012 0.003375" rpy="0 0 ${PI/2}" />
+            <geometry>
+                <box size="0.064 0.0465 0.04525" />
             </geometry>
         </collision>
@@ -173,7 +173,7 @@
         </visual>
         <collision>
-            <origin xyz="0 0 0" rpy="0 0 0" />
-            <geometry>
-                <mesh filename="file://$(find niryo_robot_description)/meshes/ned3pro/stl/hand_link.STL" />
+            <origin xyz="-6.10156e-06 0 0.0085" rpy="0 0 0" />
+            <geometry>
+                <box size="0.0204878 0.0204366 0.038" />
             </geometry>
         </collision>
@@ -194,7 +194,7 @@
         </visual>
         <collision>
-            <origin xyz="0 0 0" rpy="0 0 0" />
-            <geometry>
-                <mesh filename="file://$(find niryo_robot_description)/meshes/ned3pro/stl/niryo_scoop_v4-ros.STL" scale="0.001 0.001 0.001" />
+            <origin xyz="0.0822998 1.1301e-06 -0.0552548" rpy="0 0 0" />
+            <geometry>
+                <box size="0.1854 0.054 0.11051" />
             </geometry>
         </collision>
